File: Hardware/Power.sch (KiCad schematic (older format))
At the start: 0 parts

Commit message: power
Parts:
- added C1, C2: 1uF, symbol Device:C
- added U2: LM1117-3.3, symbol Regulator_Linear:LM1117-3.3
Connections:
- new net +3V3: C2.1, U2.2 (VO)
- new net +5V: C1.1, U2.3 (VI)
- new net GND: C1.2, C2.2, U2.1 (GND)
Changed lines of the file:
@@
 encoding utf-8
 Sheet 3 3
-Title ""
+Title "Power scheme"
 Date ""
 Rev ""
-Comp ""
+Comp "Konrad Borowik"
 Comment1 ""
 Comment2 ""
@@
 Comment4 ""
 $EndDescr
+$Comp
+L Regulator_Linear:LM1117-3.3 U2
+U 1 1 61AAF6E5
+P 5300 3600
+F 0 "U2" H 5300 3842 50  0000 C CNN
+F 1 "LM1117-3.3" H 5300 3751 50  0000 C CNN
+F 2 "" H 5300 3600 50  0001 C CNN
+F 3 "http://www.ti.com/lit/ds/symlink/lm1117.pdf" H 5300 3600 50  0001 C CNN
+	1    5300 3600
+	1    0    0    -1
+$EndComp
+$Comp
+L Device:C C2
+U 1 1 61AB41E3
+P 5900 3750
+F 0 "C2" H 6015 3796 50  0000 L CNN
+F 1 "1uF" H 6015 3705 50  0000 L CNN
+F 2 "" H 5938 3600 50  0001 C CNN
+F 3 "~" H 5900 3750 50  0001 C CNN
+	1    5900 3750
+	1    0    0    -1
+$EndComp
+$Comp
+L Device:C C1
+U 1 1 61AB4D83
+P 4650 3750
+F 0 "C1" H 4765 3796 50  0000 L CNN
+F 1 "1uF" H 4765 3705 50  0000 L CNN
+F 2 "" H 4688 3600 50  0001 C CNN
+F 3 "~" H 4650 3750 50  0001 C CNN
+	1    4650 3750
+	1    0    0    -1
+$EndComp
+Wire Wire Line
+	5900 3600 5600 3600
+Wire Wire Line
+	5000 3600 4650 3600
+Wire Wire Line
+	4650 3900 4650 4050
+Wire Wire Line
+	4650 4050 5300 4050
+Wire Wire Line
+	5300 4050 5300 3900
+Wire Wire Line
+	5900 3900 5900 4050
+Wire Wire Line
+	5900 4050 5300 4050
+Connection ~ 5300 4050
+Wire Wire Line
+	5300 4050 5300 4200
+$Comp
+L power:GND #PWR?
+U 1 1 61AB651C
+P 5300 4200
+F 0 "#PWR?" H 5300 3950 50  0001 C CNN
+F 1 "GND" H 5305 4027 50  0000 C CNN
+F 2 "" H 5300 4200 50  0001 C CNN
+F 3 "" H 5300 4200 50  0001 C CNN
+	1    5300 4200
+	1    0    0    -1
+$EndComp
+Wire Wire Line
+	4650 3600 4350 3600
+Wire Wire Line
+	4350 3600 4350 3550
+Connection ~ 4650 3600
+Wire Wire Line
+	6200 3550 6200 3600
+Wire Wire Line
+	6200 3600 5900 3600
+Connection ~ 5900 3600
+$Comp
+L power:+5V #PWR?
+U 1 1 61AB7127
+P 4350 3550
+F 0 "#PWR?" H 4350 3400 50  0001 C CNN
+F 1 "+5V" H 4365 3723 50  0000 C CNN
+F 2 "" H 4350 3550 50  0001 C CNN
+F 3 "" H 4350 3550 50  0001 C CNN
+	1    4350 3550
+	1    0    0    -1
+$EndComp
+$Comp
+L power:+3.3V #PWR?
+U 1 1 61AB7CD8
+P 6200 3550
+F 0 "#PWR?" H 6200 3400 50  0001 C CNN
+F 1 "+3.3V" H 6215 3723 50  0000 C CNN
+F 2 "" H 6200 3550 50  0001 C CNN
+F 3 "" H 6200 3550 50  0001 C CNN
+	1    6200 3550
+	1    0    0    -1
+$EndComp
 $EndSCHEMATC
