File: Hardware/Power.sch (KiCad schematic (older format))
At the start: 3 parts, among them U2 LM1117-3.3

Commit message: finished power scheme and some cosmetics
Parts:
- added D1: D_Zener, symbol Device:D_Zener
- added D?: LED, symbol Device:LED
- added F1: Fuse, Fuse:Fuse_0805_2012Metric_Pad1.15x1.40mm_HandSolder, symbol Device:Fuse
- added R14: 2k, symbol Device:R
- C1, C2: value 1uF -> 100nF
Connections:
- wire segments 12 -> 18
Other:
- moved on the sheet: C1, C2
Changed lines of the file:
@@
 encoding utf-8
 Sheet 3 3
-Title "Power scheme"
+Title "Power"
 Date ""
 Rev ""
@@
 L Device:C C2
 U 1 1 61AB41E3
-P 5900 3750
-F 0 "C2" H 6015 3796 50  0000 L CNN
-F 1 "1uF" H 6015 3705 50  0000 L CNN
-F 2 "" H 5938 3600 50  0001 C CNN
-F 3 "~" H 5900 3750 50  0001 C CNN
-	1    5900 3750
+P 5700 3750
+F 0 "C2" H 5815 3796 50  0000 L CNN
+F 1 "100nF" H 5815 3705 50  0000 L CNN
+F 2 "" H 5738 3600 50  0001 C CNN
+F 3 "~" H 5700 3750 50  0001 C CNN
+	1    5700 3750
 	1    0    0    -1
 $EndComp
@@
 L Device:C C1
 U 1 1 61AB4D83
-P 4650 3750
-F 0 "C1" H 4765 3796 50  0000 L CNN
-F 1 "1uF" H 4765 3705 50  0000 L CNN
-F 2 "" H 4688 3600 50  0001 C CNN
-F 3 "~" H 4650 3750 50  0001 C CNN
-	1    4650 3750
+P 4700 3750
+F 0 "C1" H 4815 3796 50  0000 L CNN
+F 1 "100nF" H 4815 3705 50  0000 L CNN
+F 2 "" H 4738 3600 50  0001 C CNN
+F 3 "~" H 4700 3750 50  0001 C CNN
+	1    4700 3750
 	1    0    0    -1
 $EndComp
 Wire Wire Line
-	5900 3600 5600 3600
+	5000 3600 4700 3600
 Wire Wire Line
-	5000 3600 4650 3600
-Wire Wire Line
-	4650 3900 4650 4050
-Wire Wire Line
-	4650 4050 5300 4050
+	4700 3900 4700 4050
 Wire Wire Line
 	5300 4050 5300 3900
 Wire Wire Line
-	5900 3900 5900 4050
-Wire Wire Line
-	5900 4050 5300 4050
+	5700 3900 5700 4050
 Connection ~ 5300 4050
 Wire Wire Line
@@
 $EndComp
 Wire Wire Line
-	4650 3600 4350 3600
-Wire Wire Line
-	4350 3600 4350 3550
-Connection ~ 4650 3600
-Wire Wire Line
-	6200 3550 6200 3600
-Wire Wire Line
-	6200 3600 5900 3600
-Connection ~ 5900 3600
+	6550 3550 6550 3600
 $Comp
 L power:+5V #PWR?
 U 1 1 61AB7127
-P 4350 3550
-F 0 "#PWR?" H 4350 3400 50  0001 C CNN
-F 1 "+5V" H 4365 3723 50  0000 C CNN
-F 2 "" H 4350 3550 50  0001 C CNN
-F 3 "" H 4350 3550 50  0001 C CNN
-	1    4350 3550
+P 3850 3550
+F 0 "#PWR?" H 3850 3400 50  0001 C CNN
+F 1 "+5V" H 3865 3723 50  0000 C CNN
+F 2 "" H 3850 3550 50  0001 C CNN
+F 3 "" H 3850 3550 50  0001 C CNN
+	1    3850 3550
 	1    0    0    -1
 $EndComp
@@
 L power:+3.3V #PWR?
 U 1 1 61AB7CD8
-P 6200 3550
-F 0 "#PWR?" H 6200 3400 50  0001 C CNN
-F 1 "+3.3V" H 6215 3723 50  0000 C CNN
-F 2 "" H 6200 3550 50  0001 C CNN
-F 3 "" H 6200 3550 50  0001 C CNN
-	1    6200 3550
+P 6550 3550
+F 0 "#PWR?" H 6550 3400 50  0001 C CNN
+F 1 "+3.3V" H 6565 3723 50  0000 C CNN
+F 2 "" H 6550 3550 50  0001 C CNN
+F 3 "" H 6550 3550 50  0001 C CNN
+	1    6550 3550
 	1    0    0    -1
 $EndComp
+$Comp
+L Device:Fuse F1
+U 1 1 61ABA2F7
+P 4100 3600
+F 0 "F1" V 3903 3600 50  0000 C CNN
+F 1 "Fuse" V 3994 3600 50  0000 C CNN
+F 2 "Fuse:Fuse_0805_2012Metric_Pad1.15x1.40mm_HandSolder" V 4030 3600 50  0001 C CNN
+F 3 "~" H 4100 3600 50  0001 C CNN
+	1    4100 3600
+	0    1    1    0
+$EndComp
+Wire Wire Line
+	3850 3550 3850 3600
+$Comp
+L Device:D_Zener D1
+U 1 1 61ABC565
+P 4350 3800
+F 0 "D1" V 4300 3600 50  0000 L CNN
+F 1 "D_Zener" V 4400 3400 50  0000 L CNN
+F 2 "" H 4350 3800 50  0001 C CNN
+F 3 "~" H 4350 3800 50  0001 C CNN
+	1    4350 3800
+	0    1    1    0
+$EndComp
+Wire Wire Line
+	4350 3650 4350 3600
+Wire Wire Line
+	4350 3600 4250 3600
+Connection ~ 4350 3600
+Wire Wire Line
+	4350 3950 4350 4050
+$Comp
+L Device:LED D?
+U 1 1 61AC0656
+P 6200 3750
+F 0 "D?" V 6239 3632 50  0000 R CNN
+F 1 "LED" V 6148 3632 50  0000 R CNN
+F 2 "" H 6200 3750 50  0001 C CNN
+F 3 "~" H 6200 3750 50  0001 C CNN
+	1    6200 3750
+	0    -1   -1   0
+$EndComp
+$Comp
+L Device:R R14
+U 1 1 61AC2812
+P 6200 4050
+F 0 "R14" H 6270 4096 50  0000 L CNN
+F 1 "2k" H 6270 4005 50  0000 L CNN
+F 2 "" V 6130 4050 50  0001 C CNN
+F 3 "~" H 6200 4050 50  0001 C CNN
+	1    6200 4050
+	1    0    0    -1
+$EndComp
+$Comp
+L power:GND #PWR?
+U 1 1 61AC3D3A
+P 6200 4200
+F 0 "#PWR?" H 6200 3950 50  0001 C CNN
+F 1 "GND" H 6205 4027 50  0000 C CNN
+F 2 "" H 6200 4200 50  0001 C CNN
+F 3 "" H 6200 4200 50  0001 C CNN
+	1    6200 4200
+	1    0    0    -1
+$EndComp
+Connection ~ 4700 3600
+Connection ~ 4700 4050
+Wire Wire Line
+	4700 4050 5300 4050
+Wire Wire Line
+	4350 4050 4700 4050
+Wire Wire Line
+	4350 3600 4700 3600
+Connection ~ 5700 3600
+Wire Wire Line
+	5700 3600 5600 3600
+Wire Wire Line
+	5700 4050 5300 4050
+Wire Wire Line
+	5700 3600 6200 3600
+Connection ~ 6200 3600
+Wire Wire Line
+	6200 3600 6550 3600
+Wire Wire Line
+	3850 3600 3950 3600
 $EndSCHEMATC

Commit message: changed resistor value in power scheme
Parts:
- R14: value 2k -> 470
Changed lines of the file:
@@
 P 6200 4050
 F 0 "R14" H 6270 4096 50  0000 L CNN
-F 1 "2k" H 6270 4005 50  0000 L CNN
+F 1 "470" H 6270 4005 50  0000 L CNN
 F 2 "" V 6130 4050 50  0001 C CNN
 F 3 "~" H 6200 4050 50  0001 C CNN

Commit message: RC added by pushbuttons, changed capacitors in uC supply
Parts:
- removed F1: Fuse, Fuse:Fuse_0805_2012Metric_Pad1.15x1.40mm_HandSolder, symbol Device:Fuse
- R14: value 470 -> 1k
- gave numbers to parts that had none: 1
Connections:
- wire segments 18 -> 17
Changed lines of the file:
@@
 	5300 4050 5300 4200
 $Comp
-L power:GND #PWR?
+L power:GND #PWR032
 U 1 1 61AB651C
 P 5300 4200
-F 0 "#PWR?" H 5300 3950 50  0001 C CNN
+F 0 "#PWR032" H 5300 3950 50  0001 C CNN
 F 1 "GND" H 5305 4027 50  0000 C CNN
 F 2 "" H 5300 4200 50  0001 C CNN
@@
 	6550 3550 6550 3600
 $Comp
-L power:+5V #PWR?
+L power:+5V #PWR031
 U 1 1 61AB7127
-P 3850 3550
-F 0 "#PWR?" H 3850 3400 50  0001 C CNN
-F 1 "+5V" H 3865 3723 50  0000 C CNN
-F 2 "" H 3850 3550 50  0001 C CNN
-F 3 "" H 3850 3550 50  0001 C CNN
-	1    3850 3550
+P 4150 3550
+F 0 "#PWR031" H 4150 3400 50  0001 C CNN
+F 1 "+5V" H 4165 3723 50  0000 C CNN
+F 2 "" H 4150 3550 50  0001 C CNN
+F 3 "" H 4150 3550 50  0001 C CNN
+	1    4150 3550
 	1    0    0    -1
 $EndComp
 $Comp
-L power:+3.3V #PWR?
+L power:+3.3V #PWR034
 U 1 1 61AB7CD8
 P 6550 3550
-F 0 "#PWR?" H 6550 3400 50  0001 C CNN
+F 0 "#PWR034" H 6550 3400 50  0001 C CNN
 F 1 "+3.3V" H 6565 3723 50  0000 C CNN
 F 2 "" H 6550 3550 50  0001 C CNN
@@
 	1    0    0    -1
 $EndComp
-$Comp
-L Device:Fuse F1
-U 1 1 61ABA2F7
-P 4100 3600
-F 0 "F1" V 3903 3600 50  0000 C CNN
-F 1 "Fuse" V 3994 3600 50  0000 C CNN
-F 2 "Fuse:Fuse_0805_2012Metric_Pad1.15x1.40mm_HandSolder" V 4030 3600 50  0001 C CNN
-F 3 "~" H 4100 3600 50  0001 C CNN
-	1    4100 3600
-	0    1    1    0
-$EndComp
 Wire Wire Line
-	3850 3550 3850 3600
+	4150 3550 4150 3600
 $Comp
 L Device:D_Zener D1
@@
 Wire Wire Line
 	4350 3650 4350 3600
-Wire Wire Line
-	4350 3600 4250 3600
 Connection ~ 4350 3600
 Wire Wire Line
 	4350 3950 4350 4050
 $Comp
-L Device:LED D?
+L Device:LED D3
 U 1 1 61AC0656
 P 6200 3750
-F 0 "D?" V 6239 3632 50  0000 R CNN
+F 0 "D3" V 6239 3632 50  0000 R CNN
 F 1 "LED" V 6148 3632 50  0000 R CNN
 F 2 "" H 6200 3750 50  0001 C CNN
@@
 P 6200 4050
 F 0 "R14" H 6270 4096 50  0000 L CNN
-F 1 "470" H 6270 4005 50  0000 L CNN
+F 1 "1k" H 6270 4005 50  0000 L CNN
 F 2 "" V 6130 4050 50  0001 C CNN
 F 3 "~" H 6200 4050 50  0001 C CNN
@@
 $EndComp
 $Comp
-L power:GND #PWR?
+L power:GND #PWR033
 U 1 1 61AC3D3A
 P 6200 4200
-F 0 "#PWR?" H 6200 3950 50  0001 C CNN
+F 0 "#PWR033" H 6200 3950 50  0001 C CNN
 F 1 "GND" H 6205 4027 50  0000 C CNN
 F 2 "" H 6200 4200 50  0001 C CNN
@@
 	6200 3600 6550 3600
 Wire Wire Line
-	3850 3600 3950 3600
+	4150 3600 4350 3600
 $EndSCHEMATC

Commit message: added footprints, updated CAN, annotated symbols
Parts:
- C16: renamed from C1; footprint (none) -> Capacitor_SMD:C_0603_1608Metric
- C17: renamed from C2; footprint (none) -> Capacitor_SMD:C_0603_1608Metric
- D1: renamed from D3; footprint (none) -> Diode_SMD:D_0805_2012Metric_Castellated
- D2: renamed from D1; footprint (none) -> Diode_SMD:D_SMB
- R18: renamed from R14; footprint (none) -> Resistor_SMD:R_0603_1608Metric
- U2: footprint (none) -> Package_TO_SOT_SMD:SOT-23
Changed lines of the file:
@@
 $Descr A4 11693 8268
 encoding utf-8
-Sheet 3 4
-Title "Power"
+Sheet 2 4
+Title "IMU"
 Date ""
 Rev ""
@@
 F 0 "U2" H 5300 3842 50  0000 C CNN
 F 1 "LM1117-3.3" H 5300 3751 50  0000 C CNN
-F 2 "" H 5300 3600 50  0001 C CNN
+F 2 "Package_TO_SOT_SMD:SOT-23" H 5300 3600 50  0001 C CNN
 F 3 "http://www.ti.com/lit/ds/symlink/lm1117.pdf" H 5300 3600 50  0001 C CNN
 	1    5300 3600
@@
 $EndComp
 $Comp
-L Device:C C2
+L Device:C C17
 U 1 1 61AB41E3
 P 5700 3750
-F 0 "C2" H 5815 3796 50  0000 L CNN
+F 0 "C17" H 5815 3796 50  0000 L CNN
 F 1 "100nF" H 5815 3705 50  0000 L CNN
-F 2 "" H 5738 3600 50  0001 C CNN
+F 2 "Capacitor_SMD:C_0603_1608Metric" H 5738 3600 50  0001 C CNN
 F 3 "~" H 5700 3750 50  0001 C CNN
 	1    5700 3750
@@
 $EndComp
 $Comp
-L Device:C C1
+L Device:C C16
 U 1 1 61AB4D83
 P 4700 3750
-F 0 "C1" H 4815 3796 50  0000 L CNN
+F 0 "C16" H 4815 3796 50  0000 L CNN
 F 1 "100nF" H 4815 3705 50  0000 L CNN
-F 2 "" H 4738 3600 50  0001 C CNN
+F 2 "Capacitor_SMD:C_0603_1608Metric" H 4738 3600 50  0001 C CNN
 F 3 "~" H 4700 3750 50  0001 C CNN
 	1    4700 3750
@@
 	5300 4050 5300 4200
 $Comp
-L power:GND #PWR032
+L power:GND #PWR025
 U 1 1 61AB651C
 P 5300 4200
-F 0 "#PWR032" H 5300 3950 50  0001 C CNN
+F 0 "#PWR025" H 5300 3950 50  0001 C CNN
 F 1 "GND" H 5305 4027 50  0000 C CNN
 F 2 "" H 5300 4200 50  0001 C CNN
@@
 	6550 3550 6550 3600
 $Comp
-L power:+5V #PWR031
+L power:+5V #PWR023
 U 1 1 61AB7127
 P 4150 3550
-F 0 "#PWR031" H 4150 3400 50  0001 C CNN
+F 0 "#PWR023" H 4150 3400 50  0001 C CNN
 F 1 "+5V" H 4165 3723 50  0000 C CNN
 F 2 "" H 4150 3550 50  0001 C CNN
@@
 $EndComp
 $Comp
-L power:+3.3V #PWR034
+L power:+3.3V #PWR024
 U 1 1 61AB7CD8
 P 6550 3550
-F 0 "#PWR034" H 6550 3400 50  0001 C CNN
+F 0 "#PWR024" H 6550 3400 50  0001 C CNN
 F 1 "+3.3V" H 6565 3723 50  0000 C CNN
 F 2 "" H 6550 3550 50  0001 C CNN
@@
 	4150 3550 4150 3600
 $Comp
-L Device:D_Zener D1
+L Device:D_Zener D2
 U 1 1 61ABC565
 P 4350 3800
-F 0 "D1" V 4300 3600 50  0000 L CNN
+F 0 "D2" V 4300 3600 50  0000 L CNN
 F 1 "D_Zener" V 4400 3400 50  0000 L CNN
-F 2 "" H 4350 3800 50  0001 C CNN
+F 2 "Diode_SMD:D_SMB" H 4350 3800 50  0001 C CNN
 F 3 "~" H 4350 3800 50  0001 C CNN
 	1    4350 3800
@@
 	4350 3950 4350 4050
 $Comp
-L Device:LED D3
+L Device:LED D1
 U 1 1 61AC0656
 P 6200 3750
-F 0 "D3" V 6239 3632 50  0000 R CNN
+F 0 "D1" V 6239 3632 50  0000 R CNN
 F 1 "LED" V 6148 3632 50  0000 R CNN
-F 2 "" H 6200 3750 50  0001 C CNN
+F 2 "Diode_SMD:D_0805_2012Metric_Castellated" H 6200 3750 50  0001 C CNN
 F 3 "~" H 6200 3750 50  0001 C CNN
 	1    6200 3750
@@
 $EndComp
 $Comp
-L Device:R R14
+L Device:R R18
 U 1 1 61AC2812
 P 6200 4050
-F 0 "R14" H 6270 4096 50  0000 L CNN
+F 0 "R18" H 6270 4096 50  0000 L CNN
 F 1 "1k" H 6270 4005 50  0000 L CNN
-F 2 "" V 6130 4050 50  0001 C CNN
+F 2 "Resistor_SMD:R_0603_1608Metric" V 6130 4050 50  0001 C CNN
 F 3 "~" H 6200 4050 50  0001 C CNN
 	1    6200 4050
@@
 $EndComp
 $Comp
-L power:GND #PWR033
+L power:GND #PWR026
 U 1 1 61AC3D3A
 P 6200 4200
-F 0 "#PWR033" H 6200 3950 50  0001 C CNN
+F 0 "#PWR026" H 6200 3950 50  0001 C CNN
 F 1 "GND" H 6205 4027 50  0000 C CNN
 F 2 "" H 6200 4200 50  0001 C CNN
