File: Hardware/IMU.sch (KiCad schematic (older format))
At the start: 6 parts, among them U20 IMS330DHCX

Commit message: added footprints, updated CAN, annotated symbols
Parts:
- renumbered C45 to C18, C46 to C19, FB3 to FB1, R64 to R19, R65 to R20, U20 to U3
Changed lines of the file:
@@
 $Descr A4 11693 8268
 encoding utf-8
-Sheet 4 4
-Title ""
+Sheet 3 4
+Title "IMU"
 Date ""
 Rev ""
-Comp ""
+Comp "Konrad Borowik"
 Comment1 ""
 Comment2 ""
@@
 AR Path="/61B5B7A7/61E01A5E/61AF6865" Ref="#PWR?"  Part="1"
 AR Path="/61B5B7A7/61AF6865" Ref="#PWR?"  Part="1"
-AR Path="/61AEE0B2/61AF6865" Ref="#PWR0122"  Part="1"
-AR Path="/61B14672/61AF6865" Ref="#PWR0122"  Part="1"
-F 0 "#PWR0122" H 3650 4100 50  0001 C CNN
+AR Path="/61AEE0B2/61AF6865" Ref="#PWR?"  Part="1"
+AR Path="/61B14672/61AF6865" Ref="#PWR028"  Part="1"
+F 0 "#PWR028" H 3650 4100 50  0001 C CNN
 F 1 "GND" H 3655 4177 50  0000 C CNN
 F 2 "" H 3650 4350 50  0001 C CNN
@@
 AR Path="/61B5B7A7/61E01A5E/61AF685A" Ref="C?"  Part="1"
 AR Path="/61B5B7A7/61AF685A" Ref="C?"  Part="1"
-AR Path="/61AEE0B2/61AF685A" Ref="C45"  Part="1"
-AR Path="/61B14672/61AF685A" Ref="C45"  Part="1"
-F 0 "C45" H 3592 4146 50  0000 L CNN
+AR Path="/61AEE0B2/61AF685A" Ref="C?"  Part="1"
+AR Path="/61B14672/61AF685A" Ref="C18"  Part="1"
+F 0 "C18" H 3592 4146 50  0000 L CNN
 F 1 "100nF" H 3592 4055 50  0000 L CNN
 F 2 "Capacitor_SMD:C_0603_1608Metric" H 3500 4100 50  0001 C CNN
@@
 AR Path="/61B5B7A7/61E01A5E/61AF6854" Ref="C?"  Part="1"
 AR Path="/61B5B7A7/61AF6854" Ref="C?"  Part="1"
-AR Path="/61AEE0B2/61AF6854" Ref="C46"  Part="1"
-AR Path="/61B14672/61AF6854" Ref="C46"  Part="1"
-F 0 "C46" H 3992 4146 50  0000 L CNN
+AR Path="/61AEE0B2/61AF6854" Ref="C?"  Part="1"
+AR Path="/61B14672/61AF6854" Ref="C19"  Part="1"
+F 0 "C19" H 3992 4146 50  0000 L CNN
 F 1 "100nF" H 3992 4055 50  0000 L CNN
 F 2 "Capacitor_SMD:C_0603_1608Metric" H 3900 4100 50  0001 C CNN
@@
 AR Path="/61B5B7A7/61E01A5E/61AF6848" Ref="#PWR?"  Part="1"
 AR Path="/61B5B7A7/61AF6848" Ref="#PWR?"  Part="1"
-AR Path="/61AEE0B2/61AF6848" Ref="#PWR0121"  Part="1"
-AR Path="/61B14672/61AF6848" Ref="#PWR0121"  Part="1"
-F 0 "#PWR0121" H 3500 3400 50  0001 C CNN
+AR Path="/61AEE0B2/61AF6848" Ref="#PWR?"  Part="1"
+AR Path="/61B14672/61AF6848" Ref="#PWR027"  Part="1"
+F 0 "#PWR027" H 3500 3400 50  0001 C CNN
 F 1 "+3V3" H 3515 3723 50  0000 C CNN
 F 2 "" H 3500 3550 50  0001 C CNN
@@
 	6300 4700 6300 4650
 $Comp
-L power:GND #PWR0124
+L power:GND #PWR029
 U 1 1 61AF29D3
 P 6300 4700
-F 0 "#PWR0124" H 6300 4450 50  0001 C CNN
+F 0 "#PWR029" H 6300 4450 50  0001 C CNN
 F 1 "GND" H 6305 4527 50  0000 C CNN
 F 2 "" H 6300 4700 50  0001 C CNN
@@
 SPI_CS
 $Comp
-L power:GND #PWR0123
+L power:GND #PWR030
 U 1 1 61AEEF77
 P 5600 5400
-F 0 "#PWR0123" H 5600 5150 50  0001 C CNN
+F 0 "#PWR030" H 5600 5150 50  0001 C CNN
 F 1 "GND" V 5605 5272 50  0000 R CNN
 F 2 "" H 5600 5400 50  0001 C CNN
@@
 	7050 3700 6850 3700
 $Comp
-L Sensor_Motion:LSM6DS3 U20
+L Sensor_Motion:LSM6DS3 U3
 U 1 1 61AEE84D
 P 6250 4000
-F 0 "U20" H 6894 4046 50  0000 L CNN
+F 0 "U3" H 6894 4046 50  0000 L CNN
 F 1 "IMS330DHCX" H 6894 3955 50  0000 L CNN
 F 2 "Package_LGA:LGA-14_3x2.5mm_P0.5mm_LayoutBorder3x4y" H 5850 3300 50  0001 L CNN
@@
 SCX
 $Comp
-L Device:R_Small R64
+L Device:R_Small R19
 U 1 1 61E903DC
 P 5350 5250
-F 0 "R64" V 5154 5250 50  0000 C CNN
+F 0 "R19" V 5154 5250 50  0000 C CNN
 F 1 "0R" V 5245 5250 50  0000 C CNN
 F 2 "Resistor_SMD:R_0603_1608Metric" H 5350 5250 50  0001 C CNN
@@
 $EndComp
 $Comp
-L Device:R_Small R65
+L Device:R_Small R20
 U 1 1 61E90814
 P 5350 5550
-F 0 "R65" V 5154 5550 50  0000 C CNN
+F 0 "R20" V 5154 5550 50  0000 C CNN
 F 1 "0R" V 5245 5550 50  0000 C CNN
 F 2 "Resistor_SMD:R_0603_1608Metric" H 5350 5550 50  0001 C CNN
@@
 	3500 3550 3500 3650
 $Comp
-L Device:Ferrite_Bead_Small FB3
+L Device:Ferrite_Bead_Small FB1
 U 1 1 61B18327
 P 3500 3750
-F 0 "FB3" H 3600 3796 50  0000 L CNN
+F 0 "FB1" H 3600 3796 50  0000 L CNN
 F 1 "60R@100MHz" H 3600 3705 50  0000 L CNN
 F 2 "" V 3430 3750 50  0001 C CNN

Commit message: added temp pushbutton footprint
Parts:
- FB1: footprint (none) -> Inductor_SMD:L_0603_1608Metric
Changed lines of the file:
@@
 F 0 "FB1" H 3600 3796 50  0000 L CNN
 F 1 "60R@100MHz" H 3600 3705 50  0000 L CNN
-F 2 "" V 3430 3750 50  0001 C CNN
+F 2 "Inductor_SMD:L_0603_1608Metric" V 3430 3750 50  0001 C CNN
 F 3 "~" H 3500 3750 50  0001 C CNN
 	1    3500 3750

Commit message: wip
Parts:
- U3: footprint Package_LGA:LGA-14_3x2.5mm_P0.5mm_LayoutBorder3x4y -> PUTM_Kicad_FOOTPRINTS:LGA-14_3x2.5mm_P0.5mm_LayoutBorder3x4y
Changed lines of the file:
@@
 F 0 "U3" H 6894 4046 50  0000 L CNN
 F 1 "IMS330DHCX" H 6894 3955 50  0000 L CNN
-F 2 "Package_LGA:LGA-14_3x2.5mm_P0.5mm_LayoutBorder3x4y" H 5850 3300 50  0001 L CNN
+F 2 "PUTM_Kicad_FOOTPRINTS:LGA-14_3x2.5mm_P0.5mm_LayoutBorder3x4y" H 5850 3300 50  0001 L CNN
 F 3 "www.st.com/resource/en/datasheet/lsm6ds3.pdf" H 6350 3350 50  0001 C CNN
 	1    6250 4000
