File: Hardware/Pushbuttons.sch (KiCad schematic (older format))
At the start: 16 parts, among them SW3 SW_Push, SW4 SW_Push, SW5 SW_Push, SW6 SW_Push

Commit message: added more buttons
Parts:
- added C31, C32, C33, C34: 100nF, Capacitor_SMD:C_0603_1608Metric, symbol Device:C
- added R34, R35, R36, R37: 1k, Resistor_SMD:R_0603_1608Metric, symbol Device:R
- added R38, R39, R40, R41: 10k, Resistor_SMD:R_0603_1608Metric, symbol Device:R
- added SW10, SW11, SW8, SW9: SW_Push, Button_Switch_THT:MyPushbuttonSwitch, symbol Switch:SW_Push
Connections:
- net +3V3: now also SW10.1, SW11.1, SW8.1, SW9.1
- net GND: now also C31.2, C32.2, C33.2, C34.2, R38.1, R39.1, R40.1, R41.1
- new net: R34.2, SW8.2
- new net: R35.2, SW9.2
- new net: R36.2, SW10.2
- new net: R37.2, SW11.2
- new net SW10: C34.1, R37.1, R41.2
- new net SW7: C31.1, R34.1, R38.2
- new net SW8: C32.1, R35.1, R39.2
- new net SW9: C33.1, R36.1, R40.2
Other:
- moved on the sheet: C15, C3, C5, C6, R12, R13, R14, R15, R16, R17, R26, R27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

Commit message: changed positions for buttons
Parts:
- renumbered SW11 to SW10, SW8 to SW7, SW9 to SW8, SW10 to SW9
Changed lines of the file:
@@
 Connection ~ 4400 3300
 $Comp
-L Switch:SW_Push SW8
+L Switch:SW_Push SW7
 U 1 1 62A460B2
 P 4950 4500
-F 0 "SW8" H 4950 4785 50  0000 C CNN
+F 0 "SW7" H 4950 4785 50  0000 C CNN
 F 1 "SW_Push" H 4950 4694 50  0000 C CNN
 F 2 "Button_Switch_THT:MyPushbuttonSwitch" H 4950 4700 50  0001 C CNN
@@
 $EndComp
 $Comp
-L Switch:SW_Push SW9
+L Switch:SW_Push SW8
 U 1 1 62A460B8
 P 4950 5100
-F 0 "SW9" H 4950 5385 50  0000 C CNN
+F 0 "SW8" H 4950 5385 50  0000 C CNN
 F 1 "SW_Push" H 4950 5294 50  0000 C CNN
 F 2 "Button_Switch_THT:MyPushbuttonSwitch" H 4950 5300 50  0001 C CNN
@@
 Connection ~ 4400 4500
 $Comp
-L Switch:SW_Push SW10
+L Switch:SW_Push SW9
 U 1 1 62A7A9E2
 P 4950 5700
-F 0 "SW10" H 4950 5985 50  0000 C CNN
+F 0 "SW9" H 4950 5985 50  0000 C CNN
 F 1 "SW_Push" H 4950 5894 50  0000 C CNN
 F 2 "Button_Switch_THT:MyPushbuttonSwitch" H 4950 5900 50  0001 C CNN
@@
 $EndComp
 $Comp
-L Switch:SW_Push SW11
+L Switch:SW_Push SW10
 U 1 1 62A7A9E8
 P 4950 6300
-F 0 "SW11" H 4950 6585 50  0000 C CNN
+F 0 "SW10" H 4950 6585 50  0000 C CNN
 F 1 "SW_Push" H 4950 6494 50  0000 C CNN
 F 2 "Button_Switch_THT:MyPushbuttonSwitch" H 4950 6500 50  0001 C CNN
