File: Hardware/_autosave-KieraV2.kicad_pcb (KiCad board)
At the start: 2 copper layers, 111 x 63.2 mm, 113 parts, among them J1 Conn_01x04_Male, J2 Conn_01x06_Male, SW1 SW_Rotary2x4, SW10 SW_Push, SW11 SW_MEC_5G, SW2 SW_Rotary2x4, SW3 SW_Push, SW4 SW_Push, SW5 SW_Push, SW6 SW_Push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

Commit message: updated pcb
Routing:
- net safe5V: track 63.4 -> 64.6 mm
- net GND: vias 280 -> 281
Changed lines of the file:
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@@
   (via (at 147.86 139.69) (size 0.8) (drill 0.4) (layers F.Cu B.Cu) (net 1))
   (via (at 146.41 138.365) (size 0.8) (drill 0.4) (layers F.Cu B.Cu) (net 1))
-  (via (at 147.435 135.29) (size 0.8) (drill 0.4) (layers F.Cu B.Cu) (net 1))
   (via (at 132.6 144.15) (size 0.8) (drill 0.4) (layers F.Cu B.Cu) (net 1))
   (via (at 128.95 144.075) (size 0.8) (drill 0.4) (layers F.Cu B.Cu) (net 1))
@@
   (via (at 142.38 127.91) (size 0.8) (drill 0.4) (layers F.Cu B.Cu) (net 1))
   (via (at 183.57 110.31) (size 0.8) (drill 0.4) (layers F.Cu B.Cu) (net 1))
+  (via (at 146.23 132.81) (size 0.8) (drill 0.4) (layers F.Cu B.Cu) (net 1))
+  (via (at 146.65 123.3) (size 0.8) (drill 0.4) (layers F.Cu B.Cu) (net 1))
   (segment (start 152.525 104.775) (end 152.85 105.1) (width 0.25) (layer F.Cu) (net 2))
   (segment (start 151.05 104.775) (end 152.525 104.775) (width 0.25) (layer F.Cu) (net 2))
@@
   (segment (start 138.585 128.04) (end 138.51 127.965) (width 1) (layer F.Cu) (net 100))
   (segment (start 138.585 130.16) (end 138.585 128.04) (width 1) (layer F.Cu) (net 100))
-  (via (at 145.6 133.42) (size 0.8) (drill 0.4) (layers F.Cu B.Cu) (net 101))
-  (segment (start 144.855 133.42) (end 145.6 133.42) (width 1) (layer F.Cu) (net 101))
-  (segment (start 143.21 131.775) (end 144.855 133.42) (width 1) (layer F.Cu) (net 101))
-  (segment (start 143.21 130.375) (end 143.21 131.775) (width 1) (layer F.Cu) (net 101))
-  (segment (start 174.625 116.8) (end 174.625 114.4) (width 1) (layer B.Cu) (net 101))
-  (segment (start 158.005 133.42) (end 174.625 116.8) (width 1) (layer B.Cu) (net 101))
-  (segment (start 145.6 133.42) (end 158.005 133.42) (width 1) (layer B.Cu) (net 101))
+  (via (at 145.67 134.66) (size 0.8) (drill 0.4) (layers F.Cu B.Cu) (net 101))
+  (segment (start 143.21 132.2) (end 145.67 134.66) (width 1) (layer F.Cu) (net 101))
+  (segment (start 143.21 130.375) (end 143.21 132.2) (width 1) (layer F.Cu) (net 101))
+  (segment (start 174.625 116.8) (end 156.765 134.66) (width 1) (layer B.Cu) (net 101))
+  (segment (start 174.625 114.4) (end 174.625 116.8) (width 1) (layer B.Cu) (net 101))
+  (segment (start 156.765 134.66) (end 145.67 134.66) (width 1) (layer B.Cu) (net 101))
   (zone (net 1) (net_name GND) (layer F.Cu) (hatch edge 0.508)
     (connect_pads (clearance 0.508))
